File: RPi UART-USB Shim.brd (EAGLE design)
At the start: 19.1 x 12.7 mm, 14 parts, among them U1 CP2104

Commit message: Completed board layout and clenaed up schematic
Parts:
- added U2: NUF2030XV6, on-semiconductor:SOT-563
- moved C4 2.54 mm to (9.21, 11.7)
- moved C3 1.31 mm to (14.0, 6.67)
- moved C2 1.31 mm to (14.0, 5.71)
- moved D2 1.27 mm to (18.1, 7.62)
- moved R3 1.27 mm to (16.8, 7.62)
- moved C1 0.71 mm to (14.0, 8.26)
- moved R1 0.45 mm to (14.0, 9.21)
- moved U1 0.32 mm to (10.2, 8.89)
Connections:
- new net D+.RAW: U2.3, USB1.3
- new net D-.RAW: U2.1, USB1.2
- net D+: now also U2.4; no longer USB1.3
- net D-: now also U2.6; no longer USB1.2
- net GND: now also U2.2
- net VIN: now also U2.5
Routing:
- net VDDIO: track 0.00 -> 19.4 mm, vias 0 -> 5
- net N$8: track 0.00 -> 16.3 mm, vias 0 -> 2
- net VIN: track 0.00 -> 13.5 mm, vias 0 -> 2
- net N$4: track 0.00 -> 8.58 mm
- net N$5: track 0.00 -> 8.07 mm
- net PI_TXO: track 0.00 -> 8.03 mm, vias 0 -> 1
- net D-: track 0.00 -> 8.00 mm, vias 0 -> 2
- net D+: track 0.00 -> 7.95 mm, vias 0 -> 2
- net PI_RXI: track 0.00 -> 7.75 mm, vias 0 -> 1
- net D+.RAW: track 0.00 -> 4.19 mm
- net D-.RAW: track 0.00 -> 4.08 mm
- net GND: track 0.00 -> 2.26 mm, vias 0 -> 4
- net N$2: track 0.00 -> 1.55 mm
- net N$7: track 0.00 -> 1.27 mm
- net N$6: track 0.00 -> 1.27 mm
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Other:
- board text added: "Cruz Monrreal II"
- board text added: "RPi UART USB Shim"
