File: RPi UART-USB Shim.sch (EAGLE design)
At the start: 14 parts, among them U1 CP2104

Commit message: Completed board layout and clenaed up schematic
Parts:
- added U2: NUF2030XV6, on-semiconductor:NUF2030XV6
Connections:
- new net D+.RAW: U2.D2.I, USB1.D+
- new net D-.RAW: U2.D1.I, USB1.D-
- net D+: now also U2.D2.O; no longer USB1.D+
- net D-: now also U2.D1.O; no longer USB1.D-
- net GND: now also U2.GND
- net VIN: now also U2.VBUS
Other:
- note added: "RPi UART Connector"
- note added: "USB Connector w/ ESD Protection"
- note added: "USB to UART Converter"
- moved on the sheet: C1, C2, C3, C4, D1, D2, D3, H1, R1, R2, R3, R4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
